File: classic/hw/v1/classic-v1.sch (KiCad schematic (older format))
At the start: 14 parts, among them J1 ISP, J2 USB, SW1 ESWITCH, U1 ATTINY85, U2 LDO

Commit message: hw+
Parts:
- C1, C4: symbol CP1 -> classic-v1-rescue:CP1
- C2, C3: symbol C -> classic-v1-rescue:C
- D1: symbol LED -> classic-v1-rescue:LED
- J1: symbol ISP -> classic-v1-rescue:ISP
- J2: symbol USB -> classic-v1-rescue:USB
- R1, R2, R3, R4: symbol R -> classic-v1-rescue:R
- SW1: symbol ESWITCH -> classic-v1-rescue:ESWITCH
- U1: symbol ATTINY85 -> classic-v1-rescue:ATTINY85
- U2: symbol LDO -> classic-v1-rescue:LDO
Changed lines of the file:
@@
-EESchema Schematic File Version 2
-LIBS:microjelly
-LIBS:device
-LIBS:beeon-classic-cache
-EELAYER 27 0
+EESchema Schematic File Version 4
+EELAYER 30 0
 EELAYER END
 $Descr A4 11693 8268
@@
 $EndDescr
 $Comp
-L ATTINY85 U1
+L classic-v1-rescue:ATTINY85 U1
 U 1 1 53F78C6C
 P 4000 3550
@@
 $EndComp
 $Comp
-L LDO U2
+L classic-v1-rescue:LDO U2
 U 1 1 53F78C7B
 P 8500 2000
@@
 $EndComp
 $Comp
-L USB J2
+L classic-v1-rescue:USB J2
 U 1 1 53F78CBD
 P 9200 4000
@@
 $EndComp
 $Comp
-L ISP J1
+L classic-v1-rescue:ISP J1
 U 1 1 53F78CDD
 P 8500 5750
@@
 $EndComp
 $Comp
-L ESWITCH SW1
+L classic-v1-rescue:ESWITCH SW1
 U 1 1 53F78CF3
 P 4150 6750
@@
 $EndComp
 $Comp
-L CP1 C1
+L classic-v1-rescue:CP1 C1
 U 1 1 53F78D86
 P 3000 3800
@@
 $EndComp
 $Comp
-L R R1
+L classic-v1-rescue:R R1
 U 1 1 53F78DA1
 P 1850 6800
@@
 $EndComp
 $Comp
-L LED D1
+L classic-v1-rescue:LED D1
 U 1 1 53F78DB1
 P 2400 6800
@@
 $EndComp
 $Comp
-L C C3
+L classic-v1-rescue:C C3
 U 1 1 53F78DE2
 P 8500 2500
@@
 	9050 2500 9050 2150
 Wire Wire Line
-	7700 2500 8300 2500
-Wire Wire Line
-	7950 2000 7950 2500
+	7700 2500 7950 2500
+Wire Wire Line
+	7950 2000 7950 2150
 Connection ~ 7950 2150
 $Comp
-L C C2
+L classic-v1-rescue:C C2
 U 1 1 53F78E1D
 P 7700 2300
@@
 Connection ~ 7950 2500
 Wire Wire Line
-	7700 1500 7700 2100
+	7700 1500 7700 1850
 Wire Wire Line
 	7700 1850 7950 1850
@@
 	7700 2700 7700 2500
 $Comp
-L CP1 C4
+L classic-v1-rescue:CP1 C4
 U 1 1 53F78E77
 P 9200 2050
@@
 $EndComp
 Wire Wire Line
-	9050 1850 9450 1850
+	9050 1850 9200 1850
 Wire Wire Line
 	9200 2250 9200 2700
@@
 Connection ~ 9200 1850
 Wire Wire Line
-	7700 2700 9500 2700
+	7700 2700 9200 2700
 Connection ~ 9200 2700
 Text GLabel 9450 1500 2    60   Input ~ 0
@@
 	8550 4050 8850 4050
 $Comp
-L R R4
+L classic-v1-rescue:R R4
 U 1 1 53F78F69
 P 8500 3950
@@
 	8250 4250 8250 3950
 $Comp
-L R R3
+L classic-v1-rescue:R R3
 U 1 1 53F78FA1
 P 8500 3800
@@
 $EndComp
 $Comp
-L R R2
+L classic-v1-rescue:R R2
 U 1 1 53F78FA7
 P 8500 3650
@@
 	7950 3650 8250 3650
 Wire Wire Line
-	2800 4000 3250 4000
+	2800 4000 3000 4000
 Text GLabel 2800 4000 0    60   Input ~ 0
 GND
@@
 	3250 3600 3250 3700
 Wire Wire Line
-	2800 3600 3250 3600
+	2800 3600 3000 3600
 Text GLabel 2800 3600 0    60   Input ~ 0
 VCC
@@
 PB2
 Wire Wire Line
-	3550 6650 4650 6650
-Wire Wire Line
-	3650 6850 4750 6850
+	3550 6650 3650 6650
+Wire Wire Line
+	3650 6850 4650 6850
 Connection ~ 3650 6650
 Connection ~ 4650 6850
+Wire Wire Line
+	7950 2150 7950 2500
+Wire Wire Line
+	7950 2500 8300 2500
+Wire Wire Line
+	9200 1850 9450 1850
+Wire Wire Line
+	9200 2700 9500 2700
+Wire Wire Line
+	7700 1850 7700 2100
+Wire Wire Line
+	3000 4000 3250 4000
+Wire Wire Line
+	3000 3600 3250 3600
+Wire Wire Line
+	3650 6650 4650 6650
+Wire Wire Line
+	4650 6850 4750 6850
 $EndSCHEMATC
